File: newk-tabesque48.kicad_pcb (KiCad board)
At the start: 2 copper layers, 192.5 x 118.4 mm, 98 parts, among them SW1 SW_Push, U1 ProMicro

Commit message: created gerber
Routing:
- net Net-(D42-A): track 0.00 -> 13.6 mm
- net Net-(D40-A): track 0.00 -> 13.6 mm
- net Net-(D41-A): track 0.00 -> 13.6 mm
- net Net-(D43-A): track 0.00 -> 13.5 mm

Commit message: work and stuff i don't remember lots of fusion
Other:
- outline, holes or cut-outs redrawn
- board text added: "tabesco-48"
Changed lines of the file:
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@@
 	)
 	(gr_arc
-		(start 58.928 27.305)
-		(mid 59.22558 26.58658)
-		(end 59.944 26.289)
+		(start 58.928 48.387)
+		(mid 59.22558 47.66858)
+		(end 59.944 47.371)
+		(stroke
+			(width 0.05)
+			(type default)
+		)
+		(layer "Edge.Cuts")
+	)
+	(gr_line
+		(start 208.834 26.287)
+		(end 250.444 26.289)
+		(stroke
+			(width 0.05)
+			(type default)
+		)
+		(layer "Edge.Cuts")
+	)
+	(gr_line
+		(start 208.153989 26.537265)
+		(end 187.574 47.117)
 		(stroke
 			(width 0.05)
@@
 		(start 251.46 27.305)
 		(end 251.46 143.637)
-		(stroke
-			(width 0.05)
-			(type default)
-		)
-		(layer "Edge.Cuts")
-	)
-	(gr_line
-		(start 58.928 143.637)
-		(end 58.928 27.305)
 		(stroke
 			(width 0.05)
@@
 		(layer "Edge.Cuts")
 	)
-	(gr_line
-		(start 250.444 26.289)
-		(end 59.944 26.289)
+	(gr_arc
+		(start 208.153989 26.537265)
+		(mid 208.468943 26.344063)
+		(end 208.834 26.287)
+		(stroke
+			(width 0.05)
+			(type default)
+		)
+		(layer "Edge.Cuts")
+	)
+	(gr_arc
+		(start 187.574 47.117)
+		(mid 187.259046 47.310202)
+		(end 186.893989 47.367265)
 		(stroke
 			(width 0.05)
@@
 		(start 59.944 144.653)
 		(end 250.444 144.653)
+		(stroke
+			(width 0.05)
+			(type default)
+		)
+		(layer "Edge.Cuts")
+	)
+	(gr_line
+		(start 58.928 48.387)
+		(end 58.928 143.637)
+		(stroke
+			(width 0.05)
+			(type default)
+		)
+		(layer "Edge.Cuts")
+	)
+	(gr_line
+		(start 59.944 47.371)
+		(end 186.893989 47.367265)
 		(stroke
 			(width 0.05)
@@
 		(layer "Edge.Cuts")
 	)
+	(gr_text "tabesco-48"
+		(at 155.067 100.457 0)
+		(layer "F.SilkS")
+		(effects
+			(font
+				(size 75 21)
+				(thickness 5.25)
+				(bold yes)
+			)
+		)
+	)
 	(segment
