File: newk-tabesque48.kicad_sch (KiCad schematic)
At the start: 98 parts, among them SW1 SW_Push, U1 ProMicro

Commit message: created tabasco slide verson
Connections:
- net col0: now also U1.1 (D3-TX); no longer U1.11 (B4)
- net col1: now also U1.13 (B0); no longer U1.12 (B5)
- net row0: now also U1.8 (C6); no longer U1.10 (E6)
- net row2: now also U1.10 (E6); no longer U1.8 (C6)
- net row3: now also U1.11 (B4); no longer U1.7 (D4)
- net row4: now also U1.12 (B5); no longer U1.6 (D0)
- net col_tmo: no longer names the net of U1.5 (D1)
Changed lines of the file:
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@@
 	)
 	(label "col1"
-		(at 24.13 49.53 180)
-		(fields_autoplaced yes)
-		(effects
-			(font
-				(size 1.27 1.27)
-			)
-			(justify right bottom)
+		(at 49.53 21.59 0)
+		(fields_autoplaced yes)
+		(effects
+			(font
+				(size 1.27 1.27)
+			)
+			(justify left bottom)
 		)
 	)
@@
 	)
 	(label "row0"
-		(at 24.13 44.45 180)
-		(fields_autoplaced yes)
-		(effects
-			(font
-				(size 1.27 1.27)
-			)
-			(justify right bottom)
-		)
-	)
-	(label "col_tmo"
-		(at 24.13 31.75 180)
+		(at 24.13 39.37 180)
 		(fields_autoplaced yes)
 		(effects
@@
 	)
 	(label "row3"
-		(at 24.13 36.83 180)
+		(at 24.13 46.99 180)
 		(fields_autoplaced yes)
 		(effects
@@
 	)
 	(label "row2"
-		(at 24.13 39.37 180)
+		(at 24.13 44.45 180)
 		(fields_autoplaced yes)
 		(effects
@@
 	)
 	(label "col0"
-		(at 24.13 46.99 180)
+		(at 24.13 21.59 180)
 		(fields_autoplaced yes)
 		(effects
@@
 	)
 	(label "row4"
-		(at 24.13 34.29 180)
-		(fields_autoplaced yes)
-		(effects
+		(at 24.13 49.53 180)
+		(fields_autoplaced yes)
+		(effects
