File: newk-tabesque48.kicad_sch (KiCad schematic)
At the start: 98 parts, among them SW1 SW_Push, U1 ProMicro

Commit message: 5u
Parts:
- removed D10, D16, D17, D18, D19, D20, D24, D26, D27, D28, D29, D31, D33, D34, D35, D36, D37, D38, D39, D40, D41, D42, D43, D44, D45, D46, D47, D48, D6, D7, D8, D9: D_Small, Diode_SMD:D_SOD-123, symbol Device:D_Small
- removed MX10, MX16, MX17, MX18, MX19, MX20, MX24, MX26, MX27, MX28, MX29, MX31, MX33, MX34, MX35, MX36, MX37, MX38, MX39, MX40, MX41, MX42, MX43, MX44, MX45, MX46, MX47, MX48, MX6, MX7, MX8, MX9: MX_SW_HS, marbastlib-mx:SW_MX_HS_CPG151101S11_1u, symbol marbastlib-mx:MX_SW_HS_CPG151101S11
- removed SW1: SW_Push, Button_Switch_THT:SW_Tactile_Straight_KSA0Axx1LFTR, symbol Switch:SW_Push
- renumbered D15 to D10, D21 to D11, D22 to D12, D23 to D13, D25 to D14, D30 to D15, D32 to D16, D11 to D6, D12 to D7, D13 to D8, D14 to D9, MX15 to MX10, MX21 to MX11, MX22 to MX12, MX23 to MX13, MX25 to MX14, MX30 to MX15, MX32 to MX16, MX11 to MX6, MX12 to MX7, MX13 to MX8, MX14 to MX9
Connections:
- net col0: no longer U1.11 (B4)
- net col1: no longer U1.12 (B5)
- net col2: no longer U1.17 (F4)
- net col3: no longer U1.18 (F5)
- net col4: no longer U1.19 (F6)
- net col5: no longer U1.20 (F7)
- net col6: no longer U1.21 (B1)
- net col7: no longer U1.22 (B3)
- net col8: no longer U1.23 (B2)
- net col9: no longer U1.24 (B6)
- net col_tmo: no longer U1.5 (D1)
- net row0: no longer U1.10 (E6)
- net row1: no longer U1.9 (D7)
- net row2: no longer U1.8 (C6)
- net row3: no longer U1.7 (D4)
- net row4: no longer U1.6 (D0)
- net RST: no longer names the net of U1.15 (RST)
