File: tabesco-48.kicad_sch (KiCad schematic)
At the start: 98 parts, among them SW1 SW_Push, U1 ProMicro

Commit message: created 6 key tapdance pad 2007 rot brains stupid
Parts:
- removed D10, D13, D14, D15, D16, D17, D18, D19, D20, D23, D24, D25, D26, D27, D28, D29, D3, D30, D31, D32, D33, D34, D35, D36, D37, D38, D39, D4, D40, D41, D42, D43, D44, D45, D46, D47, D48, D5, D6, D7, D8, D9: D_Small, Diode_SMD:D_SOD-123, symbol Device:D_Small
- removed MX10, MX13, MX14, MX15, MX16, MX17, MX18, MX19, MX20, MX23, MX24, MX25, MX26, MX27, MX28, MX29, MX3, MX30, MX31, MX32, MX33, MX34, MX35, MX36, MX37, MX38, MX39, MX4, MX40, MX41, MX42, MX43, MX44, MX45, MX46, MX47, MX48, MX5, MX6, MX7, MX8, MX9: MX_SW_HS, marbastlib-mx:SW_MX_HS_CPG151101S11_1u, symbol marbastlib-mx:MX_SW_HS_CPG151101S11
- renumbered D11 to D3, D12 to D4, D21 to D5, D22 to D6, MX11 to MX3, MX12 to MX4, MX21 to MX5, MX22 to MX6
Connections:
- net col2 is gone; now on net row2: U1.17 (F4)
- net col3 is gone; now on net row1: U1.18 (F5)
- net col4 is gone; now on net row0: U1.19 (F6)
- net col8 is gone; now on net col1: U1.23 (B2)
- net col9 is gone; now on net col0: U1.24 (B6)
- net col0: no longer U1.11 (B4)
- net col1: no longer U1.12 (B5)
- net row0: no longer U1.10 (E6)
- net row1: no longer U1.9 (D7)
- net row2: no longer U1.8 (C6)
- net col5: no longer names the net of U1.20 (F7)
- net col6: no longer names the net of U1.21 (B1)
- net col7: no longer names the net of U1.22 (B3)
- net row3: no longer names the net of U1.7 (D4)
- net row4: no longer names the net of U1.6 (D0)
