File: tabesco-48.kicad_sch (KiCad schematic)
At the start: 98 parts, among them SW1 SW_Push, U1 ProMicro

Commit message: created tabesco-31
Parts:
- removed D20, D32, D33, D34, D35, D36, D37, D38, D39, D40, D41, D42, D43, D44, D45, D46, D47, D48: D_Small, Diode_SMD:D_SOD-123, symbol Device:D_Small
- removed MX20, MX32, MX33, MX34, MX35, MX36, MX37, MX38, MX39, MX40, MX41, MX42, MX43, MX44, MX45, MX46, MX47, MX48: MX_SW_HS, marbastlib-mx:SW_MX_HS_CPG151101S11_1u, symbol marbastlib-mx:MX_SW_HS_CPG151101S11
- added D29: D_Small, Diode_SMD:D_SOD-123, symbol Device:D_Small
- added MX29: MX_SW_HS, marbastlib-mx:SW_MX_HS_CPG151101S11_1u, symbol marbastlib-mx:MX_SW_HS_CPG151101S11
- renumbered D21 to D20, D22 to D21, D23 to D22, D24 to D23, D25 to D24, D26 to D25, D27 to D26, D28 to D27, D29 to D28, MX21 to MX20, MX22 to MX21, MX23 to MX22, MX24 to MX23, MX25 to MX24, MX26 to MX25, MX27 to MX26, MX28 to MX27, MX29 to MX28
Connections:
- net col0: now also MX29.2; no longer MX30.2
- net col1: now also MX30.2; no longer MX31.2
- net col7: now also MX31.2
- net row3: now also D29.1 (K)
- net col_tmo: no longer names the net of U1.5 (D1)
- net row4: no longer names the net of U1.6 (D0)
- new net: D29.2 (A), MX29.1

Commit message: work on 31
Connections:
- net col0: now also U1.5 (D1); no longer U1.11 (B4)
- net col1: now also U1.6 (D0); no longer U1.12 (B5)
- net col2: now also U1.7 (D4); no longer U1.17 (F4)
- net col3: now also U1.8 (C6); no longer U1.18 (F5)
- net col4: now also U1.9 (D7); no longer U1.19 (F6)
- net col5: now also MX31.2, U1.10 (E6); no longer U1.20 (F7)
- net col6: now also U1.11 (B4); no longer U1.21 (B1)
- net col7: now also U1.12 (B5); no longer MX31.2, U1.22 (B3)
- net row0: now also U1.17 (F4); no longer U1.10 (E6)
- net row1: now also U1.18 (F5); no longer U1.9 (D7)
- net row2: now also U1.19 (F6); no longer U1.8 (C6)
- net row3: now also U1.20 (F7); no longer U1.7 (D4)
Other:
- moved on the sheet: D31, MX31
Changed lines of the file:
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@@
 	)
 	(junction
-		(at 119.38 68.58)
+		(at 85.09 91.44)
 		(diameter 0)
 		(color 0 0 0 0)
 	)
 	(junction
-		(at 27.94 91.44)
+		(at 119.38 68.58)
 		(diameter 0)
 		(color 0 0 0 0)
 	)
 	(junction
-		(at 20.32 105.41)
+		(at 27.94 91.44)
 		(diameter 0)
 		(color 0 0 0 0)
@@
 	)
 	(junction
-		(at 62.23 68.58)
+		(at 20.32 105.41)
 		(diameter 0)
 		(color 0 0 0 0)
 	)
 	(junction
-		(at 85.09 80.01)
+		(at 62.23 68.58)
 		(diameter 0)
 		(color 0 0 0 0)
 	)
 	(junction
-		(at 107.95 91.44)
+		(at 85.09 80.01)
 		(diameter 0)
 		(color 0 0 0 0)
@@
 	(wire
 		(pts
-			(xy 100.33 100.33) (xy 100.33 97.79)
+			(xy 77.47 100.33) (xy 77.47 97.79)
 		)
 		(stroke
@@
 	(wire
 		(pts
+			(xy 31.75 105.41) (xy 77.47 105.41)
+		)
+		(stroke
+			(width 0)
+			(type default)
+		)
+	)
+	(wire
+		(pts
 			(xy 85.09 62.23) (xy 85.09 68.58)
 		)
@@
 	(wire
 		(pts
+			(xy 19.05 105.41) (xy 20.32 105.41)
+		)
+		(stroke
+			(width 0)
+			(type default)
+		)
+	)
+	(wire
+		(pts
 			(xy 39.37 91.44) (xy 39.37 102.87)
 		)
@@
 	(wire
 		(pts
-			(xy 107.95 91.44) (xy 107.95 102.87)
+			(xy 85.09 91.44) (xy 85.09 102.87)
 		)
 		(stroke
@@
 	(wire
 		(pts
-			(xy 19.05 105.41) (xy 20.32 105.41)
-		)
-		(stroke
-			(width 0)
-			(type default)
-		)
-	)
-	(wire
-		(pts
-			(xy 100.33 97.79) (xy 102.87 97.79)
+			(xy 77.47 97.79) (xy 80.01 97.79)
 		)
 		(stroke
@@
 	(wire
 		(pts
-			(xy 31.75 105.41) (xy 100.33 105.41)
-		)
-		(stroke
-			(width 0)
-			(type default)
-		)
-	)
-	(wire
-		(pts
 			(xy 119.38 68.58) (xy 119.38 80.01)
 		)
@@
 	)
 	(label "col4"
-		(at 49.53 36.83 0)
+		(at 24.13 41.91 180)
 		(fields_autoplaced yes)
 		(effects
@@
 				(size 1.27 1.27)
 			)
-			(justify left bottom)
+			(justify right bottom)
 		)
 	)
 	(label "col5"
-		(at 49.53 39.37 0)
+		(at 24.13 44.45 180)
 		(fields_autoplaced yes)
 		(effects
@@
 				(size 1.27 1.27)
 			)
-			(justify left bottom)
+			(justify right bottom)
 		)
 	)
 	(label "col1"
-		(at 24.13 49.53 180)
+		(at 24.13 34.29 180)
 		(fields_autoplaced yes)
 		(effects
@@
 	)
 	(label "row1"
-		(at 24.13 41.91 180)
+		(at 49.53 34.29 0)
 		(fields_autoplaced yes)
 		(effects
@@
 				(size 1.27 1.27)
 			)
-			(justify right bottom)
+			(justify left bottom)
 		)
 	)
 	(label "row0"
-		(at 24.13 44.45 180)
+		(at 49.53 31.75 0)
 		(fields_autoplaced yes)
 		(effects
@@
 				(size 1.27 1.27)
 			)
-			(justify right bottom)
+			(justify left bottom)
 		)
 	)
@@
 	)
 	(label "col6"
-		(at 49.53 41.91 0)
+		(at 24.13 46.99 180)
 		(fields_autoplaced yes)
 		(effects
@@
 				(size 1.27 1.27)
 			)
-			(justify left bottom)
+			(justify right bottom)
 		)
 	)
@@
 	)
 	(label "row3"
-		(at 24.13 36.83 180)
+		(at 49.53 39.37 0)
 		(fields_autoplaced yes)
 		(effects
@@
 				(size 1.27 1.27)
 			)
-			(justify right bottom)
+			(justify left bottom)
 		)
 	)
@@
 	)
 	(label "col7"
-		(at 49.53 44.45 0)
+		(at 24.13 49.53 180)
 		(fields_autoplaced yes)
 		(effects
@@
 				(size 1.27 1.27)
 			)
-			(justify left bottom)
+			(justify right bottom)
 		)
 	)
@@
 	)
 	(label "row2"
-		(at 24.13 39.37 180)
+		(at 49.53 36.83 0)
 		(fields_autoplaced yes)
 		(effects
@@
 				(size 1.27 1.27)
 			)
-			(justify right bottom)
+			(justify left bottom)
 		)
 	)
 	(label "col0"
-		(at 24.13 46.99 180)
+		(at 24.13 31.75 180)
 		(fields_autoplaced yes)
 		(effects
@@
 	)
 	(label "col3"
-		(at 49.53 34.29 0)
+		(at 24.13 39.37 180)
 		(fields_autoplaced yes)
 		(effects
@@
 				(size 1.27 1.27)
 			)
-			(justify left bottom)
+			(justify right bottom)
 		)
 	)
 	(label "col2"
-		(at 49.53 31.75 0)
+		(at 24.13 36.83 180)
 		(fields_autoplaced yes)
 		(effects
@@
 				(size 1.27 1.27)
 			)
-			(justify left bottom)
+			(justify right bottom)
 		)
 	)
@@
 	(symbol
 		(lib_id "Device:D_Small")
-		(at 100.33 102.87 90)
+		(at 77.47 102.87 90)
 		(unit 1)
 		(exclude_from_sim no)
@@
 		(dnp no)
 		(property "Reference" "D31"
-			(at 97.536 101.346 90)
+			(at 74.676 101.346 90)
 			(effects
 				(font
@@
 		)
 		(property "Value" "D_Small"
-			(at 102.87 104.1399 90)
+			(at 80.01 104.1399 90)
 			(effects
 				(font
@@
 		)
 		(property "Footprint" "Diode_SMD:D_SOD-123"
-			(at 100.33 102.87 90)
+			(at 77.47 102.87 90)
 			(effects
 				(font
@@
 		)
 		(property "Datasheet" "~"
-			(at 100.33 102.87 90)
+			(at 77.47 102.87 90)
 			(effects
 				(font
@@
 		)
 		(property "Description" "Diode, small symbol"
-			(at 100.33 102.87 0)
+			(at 77.47 102.87 0)
 			(effects
 				(font
@@
 		)
 		(property "Sim.Device" "D"
-			(at 100.33 102.87 0)
+			(at 77.47 102.87 0)
 			(effects
 				(font
@@
 		)
 		(property "Sim.Pins" "1=K 2=A"
-			(at 100.33 102.87 0)
+			(at 77.47 102.87 0)
 			(effects
 				(font
@@
 	(symbol
 		(lib_id "marbastlib-mx:MX_SW_HS_CPG151101S11")
-		(at 105.41 100.33 0)
+		(at 82.55 100.33 0)
 		(unit 1)
 		(exclude_from_sim no)
@@
 		(fields_autoplaced yes)
 		(property "Reference" "MX31"
-			(at 105.41 95.25 0)
+			(at 82.55 95.25 0)
 			(effects
 				(font
@@
 		)
 		(property "Value" "MX_SW_HS"
-			(at 105.41 95.25 0)
+			(at 82.55 95.25 0)
 			(effects
 				(font
@@
 		)
 		(property "Footprint" "marbastlib-mx:SW_MX_HS_CPG151101S11_1u"
-			(at 105.41 100.33 0)
+			(at 82.55 100.33 0)
 			(effects
 				(font
@@
 		)
 		(property "Datasheet" "~"
-			(at 105.41 100.33 0)
+			(at 82.55 100.33 0)
 			(effects
 				(font
@@
 		)
 		(property "Description" "Push button switch, normally open, two pins, 45° tilted, Kailh CPG151101S11 for Cherry MX style switches"
-			(at 105.41 100.33 0)
+			(at 82.55 100.33 0)
 			(effects
 				(font

Commit message: tabesco31 pcb done(?)
Parts:
- removed SW1: SW_Push, Button_Switch_THT:SW_Tactile_Straight_KSA0Axx1LFTR, symbol Switch:SW_Push
Changed lines of the file:
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@@
 		)
 	)
-	(global_label "RST"
-		(shape input)
-		(at 68.58 26.67 180)
-		(fields_autoplaced yes)
-		(effects
-			(font
-				(size 1.27 1.27)
-			)
-			(justify right)
-		)
-		(property "Intersheetrefs" "${INTERSHEET_REFS}"
-			(at 62.1477 26.67 0)
-			(effects
-				(font
-					(size 1.27 1.27)
-				)
-				(justify right)
-				(hide yes)
-			)
-		)
-	)
 	(symbol
 		(lib_id "marbastlib-mx:MX_SW_HS_CPG151101S11")
@@
 	)
 	(symbol
-		(lib_id "Switch:SW_Push")
-		(at 73.66 26.67 0)
-		(unit 1)
-		(exclude_from_sim no)
-		(in_bom yes)
-		(on_board yes)
-		(dnp no)
-		(fields_autoplaced yes)
-		(property "Reference" "SW1"
-			(at 73.66 19.05 0)
-			(effects
-				(font
-					(size 1.27 1.27)
-				)
-			)
-		)
-		(property "Value" "SW_Push"
-			(at 73.66 21.59 0)
-			(effects
-				(font
-					(size 1.27 1.27)
-				)
-			)
-		)
-		(property "Footprint" "Button_Switch_THT:SW_Tactile_Straight_KSA0Axx1LFTR"
-			(at 73.66 21.59 0)
-			(effects
-				(font
-					(size 1.27 1.27)
-				)
-				(hide yes)
-			)
-		)
-		(property "Datasheet" "~"
-			(at 73.66 21.59 0)
-			(effects
-				(font
-					(size 1.27 1.27)
-				)
-				(hide yes)
-			)
-		)
-		(property "Description" "Push button switch, generic, two pins"
-			(at 73.66 26.67 0)
-			(effects
-				(font
-					(size 1.27 1.27)
-				)
-				(hide yes)
-			)
-		)
-		(pin "1"
-		)
-		(pin "2"
-		)
-		(instances
-			(project ""
-				(path "/588218a1-c895-477e-9c13-7f6d8ca7aace"
-					(reference "SW1")
-					(unit 1)
-				)
-			)
-		)
-	)
-	(symbol
 		(lib_id "Device:D_Small")
 		(at 66.04 91.44 90)
@@
 					(unit 1)
 				)
-			)
-		)
-	)
-	(symbol
-		(lib_id "power:GND")
-		(at 78.74 26.67 90)
-		(unit 1)
-		(exclude_from_sim no)
-		(in_bom yes)
-		(on_board yes)
-		(dnp no)
-		(fields_autoplaced yes)
-		(property "Reference" "#PWR05"
-			(at 85.09 26.67 0)
-			(effects
-				(font
-					(size 1.27 1.27)
-				)
-				(hide yes)
-			)
-		)
-		(property "Value" "GND"
-			(at 82.55 26.6699 90)
-			(effects
-				(font
-					(size 1.27 1.27)
-				)
-				(justify right)
-			)
-		)
-		(property "Footprint" ""
-			(at 78.74 26.67 0)
-			(effects
-				(font
-					(size 1.27 1.27)
-				)
-				(hide yes)
-			)
-		)
-		(property "Datasheet" ""
-			(at 78.74 26.67 0)
-			(effects
-				(font
-					(size 1.27 1.27)
-				)
-				(hide yes)
-			)
-		)
-		(property "Description" "Power symbol creates a global label with name \"GND\" , ground"
-			(at 78.74 26.67 0)
-			(effects
-				(font
-					(size 1.27 1.27)
-				)
-				(hide yes)
-			)
-		)
-		(pin "1"
-		)
-		(instances
-			(project "newk-tabesque48"
-				(path "/588218a1-c895-477e-9c13-7f6d8ca7aace"
-					(reference "#PWR05")
-					(unit 1)
-				)

Commit message: more work, transitioning to IC in seperate repo
Parts:
- added D31, D34: D_Small, Diode_SMD:D_SOD-123, symbol Device:D_Small
- added MX31, MX32-2, MX34: MX_SW_HS, marbastlib-mx:SW_MX_HS_CPG151101S11_1u, symbol marbastlib-mx:MX_SW_HS_CPG151101S11
- renumbered D31 to D32, MX31 to MX32
Connections:
- net col0: now also U1.24 (B6); no longer U1.5 (D1)
- net col1: now also U1.23 (B2); no longer U1.6 (D0)
- net col2: now also U1.22 (B3), MX31.2; no longer U1.7 (D4)
- net col3: now also U1.12 (B5); no longer U1.8 (C6)
- net col4: now also U1.11 (B4); no longer U1.9 (D7)
- net col5: now also MX32-2.2
- net col6: now also U1.9 (D7); no longer U1.11 (B4)
- net col7: now also U1.8 (C6); no longer U1.12 (B5)
- net col8: now also U1.7 (D4), MX34.2; no longer U1.23 (B2)
- net col9: now also U1.6 (D0); no longer U1.24 (B6)
- net row0: now also U1.20 (F7); no longer U1.17 (F4)
- net row1: now also U1.19 (F6); no longer U1.18 (F5)
- net row2: now also U1.18 (F5); no longer U1.19 (F6)
- net row3: now also U1.17 (F4), D31.1 (K), D34.1 (K); no longer U1.20 (F7)
- net at D32.2 (A), MX32.1: now also MX32-2.1
- new net: D34.2 (A), MX34.1
- new net: D31.2 (A), MX31.1

Commit message: brain mode
Connections:
- net col0: now also U1.19 (F6); no longer U1.24 (B6)
- net col1: now also U1.18 (F5); no longer U1.23 (B2)
- net col2: now also U1.17 (F4); no longer U1.22 (B3)
- net col3: now also U1.6 (D0); no longer U1.12 (B5)
- net col4: now also U1.7 (D4); no longer U1.11 (B4)
- net col5: now also U1.8 (C6); no longer U1.10 (E6)
- net col6: now also U1.12 (B5); no longer U1.9 (D7)
- net col7: now also U1.11 (B4); no longer U1.8 (C6)
- net col8: now also U1.10 (E6); no longer U1.7 (D4)
- net col9: now also U1.9 (D7); no longer U1.6 (D0)
- net row0: now also U1.21 (B1); no longer U1.20 (F7)
- net row1: now also U1.22 (B3); no longer U1.19 (F6)
- net row2: now also U1.23 (B2); no longer U1.18 (F5)
- net row3: now also U1.24 (B6); no longer U1.17 (F4)
Changed lines of the file:
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@@
 	)
 	(label "col4"
-		(at 24.13 46.99 180)
+		(at 24.13 36.83 180)
 		(fields_autoplaced yes)
 		(effects
@@
 	)
 	(label "col5"
-		(at 24.13 44.45 180)
+		(at 24.13 39.37 180)
 		(fields_autoplaced yes)
 		(effects
@@
 	)
 	(label "col1"
-		(at 49.53 46.99 0)
+		(at 49.53 34.29 0)
 		(fields_autoplaced yes)
 		(effects
@@
 	)
 	(label "row1"
-		(at 49.53 36.83 0)
+		(at 49.53 44.45 0)
 		(fields_autoplaced yes)
 		(effects
@@
 	)
 	(label "row0"
-		(at 49.53 39.37 0)
+		(at 49.53 41.91 0)
 		(fields_autoplaced yes)
 		(effects
@@
 	)
 	(label "col6"
-		(at 24.13 41.91 180)
+		(at 24.13 49.53 180)
 		(fields_autoplaced yes)
 		(effects
@@
 	)
 	(label "row3"
-		(at 49.53 31.75 0)
+		(at 49.53 49.53 0)
 		(fields_autoplaced yes)
 		(effects
@@
 	)
 	(label "col7"
-		(at 24.13 39.37 180)
+		(at 24.13 46.99 180)
 		(fields_autoplaced yes)
 		(effects
@@
 	)
 	(label "col8"
-		(at 24.13 36.83 180)
+		(at 24.13 44.45 180)
 		(fields_autoplaced yes)
 		(effects
@@
 	)
 	(label "row2"
-		(at 49.53 34.29 0)
+		(at 49.53 46.99 0)
 		(fields_autoplaced yes)
 		(effects
@@
 	)
 	(label "col0"
-		(at 49.53 49.53 0)
+		(at 49.53 36.83 0)
 		(fields_autoplaced yes)
 		(effects
@@
 	)
 	(label "col3"
-		(at 24.13 49.53 180)
+		(at 24.13 34.29 180)
 		(fields_autoplaced yes)
 		(effects
@@
 	)
 	(label "col2"
-		(at 49.53 44.45 0)
+		(at 49.53 31.75 0)
 		(fields_autoplaced yes)
 		(effects
@@
 	)
 	(label "col9"
-		(at 24.13 34.29 180)
-		(fields_autoplaced yes)
-		(effects
+		(at 24.13 41.91 180)
+		(fields_autoplaced yes)
+		(effects

Commit message: finished tabesco-34
Parts:
- added D29: D_Small, Diode_SMD:D_SOD-123, symbol Device:D_Small
- added MX11-2, MX19-2, MX29: MX_SW_HS, marbastlib-mx:SW_MX_HS_CPG151101S11_1u, symbol marbastlib-mx:MX_SW_HS_CPG151101S11
- renumbered D29 to D30, D30 to D31, D31 to D32, D34 to D33, D32 to D34, MX29 to MX30, MX30 to MX31, MX31 to MX32, MX34 to MX33, MX32 to MX34, MX32-2 to MX34-2
Connections:
- net col0: now also U1.17 (F4), MX11-2.2; no longer U1.19 (F6)
- net col2: now also U1.19 (F6); no longer U1.17 (F4)
- net col3: now also MX33.2, U1.20 (F7); no longer U1.6 (D0)
- net col4: now also U1.24 (B6); no longer U1.7 (D4)
- net col5: now also U1.23 (B2); no longer MX34-2.2, MX34.2, U1.8 (C6)
- net col6: now also MX34-2.2, MX34.2, U1.22 (B3); no longer U1.12 (B5)
- net col7: now also U1.21 (B1); no longer U1.11 (B4)
- net col8: now also U1.11 (B4), MX19-2.2; no longer MX33.2, U1.10 (E6)
- net col9: now also MX29.2
- net row0: now also U1.7 (D4); no longer U1.21 (B1)
- net row1: now also U1.8 (C6); no longer U1.22 (B3)
- net row2: now also U1.10 (E6), D29.1 (K); no longer U1.23 (B2)
- net row3: now also U1.12 (B5); no longer U1.24 (B6)
- net at D11.2 (A), MX11.1: now also MX11-2.1
- net at D19.2 (A), MX19.1: now also MX19-2.1
- new net: D29.2 (A), MX29.1
Other:
- moved on the sheet: D33, D34, MX33, MX34, MX34-2

Commit message: swagbord case
Connections:
- net col0: now also MX11-2.1; no longer MX11-2.2
- net col8: now also MX19-2.1; no longer MX19-2.2
- net at D11.2 (A), MX11.1: now also MX11-2.2; no longer MX11-2.1
- net at D19.2 (A), MX19.1: now also MX19-2.2; no longer MX19-2.1
Other:
- moved on the sheet: MX11-2, MX19-2
Changed lines of the file:
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@@
 	(symbol
 		(lib_id "marbastlib-mx:MX_SW_HS_CPG151101S11")
-		(at 123.19 77.47 0)
+		(at 123.19 77.47 180)
 		(unit 1)
 		(exclude_from_sim no)
@@
 		(fields_autoplaced yes)
 		(property "Reference" "MX19-2"
-			(at 123.19 69.85 0)
+			(at 123.19 72.39 0)
 			(effects
 				(font
@@
 		)
 		(property "Value" "MX_SW_HS"
-			(at 123.19 72.39 0)
+			(at 123.19 82.55 0)
 			(effects
 				(font
@@
 	(symbol
 		(lib_id "marbastlib-mx:MX_SW_HS_CPG151101S11")
-		(at 13.97 77.47 0)
+		(at 13.97 77.47 180)
 		(unit 1)
 		(exclude_from_sim no)
@@
 		(fields_autoplaced yes)
 		(property "Reference" "MX11-2"
-			(at 13.97 69.85 0)
+			(at 13.97 72.39 0)
 			(effects
 				(font
@@
 		)
 		(property "Value" "MX_SW_HS"
-			(at 13.97 72.39 0)
+			(at 13.97 82.55 0)
 			(effects
 				(font
