File: tabesco-48.kicad_sch (KiCad schematic)
At the start: 142 parts, among them J0 AVR-ISP-6, J1 Conn_01x04, SW0 SW_Push, U1 ATmega32U4-A, U2 SRV05-4, Y0 16MHz

Commit message: prepping for kicanvas
Connections:
- net RST: now also R0.2, SW0.2, U1.13 (~{RESET})
- no-connect marks 2 -> 6
Other:
- moved on the sheet: R0, SW0
Changed lines of the file:
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@@
 	(paper "A4")
 	(junction
-		(at 57.15 62.23)
-		(diameter 0)
-		(color 0 0 0 0)
-	)
-	(junction
 		(at 187.96 275.59)
 		(diameter 0)
@@
 	)
 	(junction
+		(at 55.88 43.18)
+		(diameter 0)
+		(color 0 0 0 0)
+	)
+	(junction
 		(at 199.39 275.59)
 		(diameter 0)
@@
 	)
 	(no_connect
+		(at 87.63 64.77)
+	)
+	(no_connect
+		(at 57.15 80.01)
+	)
+	(no_connect
 		(at 104.14 106.68)
 	)
 	(no_connect
+		(at 87.63 120.65)
+	)
+	(no_connect
 		(at 129.54 101.6)
 	)
+	(no_connect
+		(at 87.63 82.55)
+	)
 	(wire
 		(pts
@@
 	(wire
 		(pts
-			(xy 58.42 62.23) (xy 57.15 62.23)
-		)
-		(stroke
-			(width 0)
-			(type default)
-		)
-	)
-	(wire
-		(pts
 			(xy 128.27 129.54) (xy 137.16 129.54)
 		)
@@
 	(wire
 		(pts
-			(xy 57.15 59.69) (xy 57.15 62.23)
-		)
-		(stroke
-			(width 0)
-			(type default)
-		)
-	)
-	(wire
-		(pts
 			(xy 180.34 280.67) (xy 182.88 280.67)
 		)
@@
 	(wire
 		(pts
+			(xy 40.64 43.18) (xy 43.18 43.18)
+		)
+		(stroke
+			(width 0)
+			(type default)
+		)
+	)
+	(wire
+		(pts
 			(xy 123.19 293.37) (xy 123.19 290.83)
 		)
@@
 	(wire
 		(pts
+			(xy 55.88 43.18) (xy 58.42 43.18)
+		)
+		(stroke
+			(width 0)
+			(type default)
+		)
+	)
+	(wire
+		(pts
 			(xy 157.48 262.89) (xy 157.48 260.35)
 		)
@@
 	(wire
 		(pts
-			(xy 58.42 49.53) (xy 58.42 52.07)
+			(xy 55.88 33.02) (xy 55.88 35.56)
 		)
 		(stroke
@@
 	(wire
 		(pts
-			(xy 57.15 62.23) (xy 57.15 64.77)
-		)
-		(stroke
-			(width 0)
-			(type default)
-		)
-	)
-	(wire
-		(pts
 			(xy 134.62 280.67) (xy 137.16 280.67)
 		)
@@
 	(wire
 		(pts
-			(xy 46.99 59.69) (xy 46.99 63.5)
-		)
-		(stroke
-			(width 0)
-			(type default)
-		)
-	)
-	(wire
-		(pts
 			(xy 67.31 275.59) (xy 67.31 285.75)
 		)
@@
 	(wire
 		(pts
-			(xy 58.42 57.15) (xy 58.42 62.23)
+			(xy 146.05 288.29) (xy 157.48 288.29)
 		)
 		(stroke
@@
 	(wire
 		(pts
-			(xy 146.05 288.29) (xy 157.48 288.29)
+			(xy 226.06 250.19) (xy 228.6 250.19)
 		)
 		(stroke
@@
 	(wire
 		(pts
-			(xy 226.06 250.19) (xy 228.6 250.19)
+			(xy 146.05 250.19) (xy 148.59 250.19)
 		)
 		(stroke
@@
 	(wire
 		(pts
-			(xy 146.05 250.19) (xy 148.59 250.19)
+			(xy 134.62 283.21) (xy 134.62 280.67)
 		)
 		(stroke
@@
 	(wire
 		(pts
-			(xy 134.62 283.21) (xy 134.62 280.67)
+			(xy 191.77 257.81) (xy 203.2 257.81)
 		)
 		(stroke
@@
 	(wire
 		(pts
-			(xy 191.77 257.81) (xy 203.2 257.81)
+			(xy 55.88 40.64) (xy 55.88 43.18)
 		)
 		(stroke
@@
 	(wire
 		(pts
+			(xy 53.34 43.18) (xy 55.88 43.18)
+		)
+		(stroke
+			(width 0)
+			(type default)
+		)
+	)
+	(wire
+		(pts
 			(xy 123.19 257.81) (xy 134.62 257.81)
 		)
@@
 		)
 	)
+	(global_label "RST"
+		(shape input)
+		(at 57.15 64.77 180)
+		(fields_autoplaced yes)
+		(effects
+			(font
+				(size 1.27 1.27)
+			)
+			(justify right)
+		)
+		(property "Intersheetrefs" "${INTERSHEET_REFS}"
+			(at 50.7177 64.77 0)
+			(effects
+				(font
+					(size 1.27 1.27)
+				)
+				(justify right)
+				(hide yes)
+			)
+		)
+	)
 	(global_label "SCK"
 		(shape input)
@@
 		)
 	)
+	(global_label "RST"
+		(shape input)
+		(at 58.42 43.18 270)
+		(fields_autoplaced yes)
+		(effects
+			(font
+				(size 1.27 1.27)
+			)
+			(justify right)
+		)
+		(property "Intersheetrefs" "${INTERSHEET_REFS}"
+			(at 58.42 49.6123 90)
+			(effects
+				(font
+					(size 1.27 1.27)
+				)
+				(justify right)
+				(hide yes)
+			)
+		)
+	)
 	(global_label "MOSI"
 		(shape input)
@@
 	(symbol
 		(lib_id "Switch:SW_Push")
-		(at 52.07 59.69 0)
+		(at 48.26 43.18 0)
 		(unit 1)
 		(exclude_from_sim no)
@@
 		(fields_autoplaced yes)
 		(property "Reference" "SW0"
-			(at 52.07 52.07 0)
+			(at 48.26 35.56 0)
 			(effects
 				(font
@@
 		)
 		(property "Value" "SW_Push"
-			(at 52.07 54.61 0)
+			(at 48.26 38.1 0)
 			(effects
 				(font
@@
 		)
 		(property "Footprint" "Button_Switch_THT:SW_Tactile_Straight_KSA0Axx1LFTR"
-			(at 52.07 54.61 0)
+			(at 48.26 38.1 0)
 			(effects
 				(font
@@
 		)
 		(property "Datasheet" "~"
-			(at 52.07 54.61 0)
+			(at 48.26 38.1 0)
 			(effects
 				(font
@@
 		)
 		(property "Description" "Push button switch, generic, two pins"
-			(at 52.07 59.69 0)
+			(at 48.26 43.18 0)
 			(effects
 				(font
@@
 	(symbol
 		(lib_id "power:+5V")
-		(at 58.42 49.53 0)
+		(at 55.88 33.02 0)
 		(unit 1)
 		(exclude_from_sim no)
@@
 		(fields_autoplaced yes)
 		(property "Reference" "#PWR04"
-			(at 58.42 53.34 0)
+			(at 55.88 36.83 0)
 			(effects
 				(font
@@
 		)
 		(property "Value" "+5V"
-			(at 58.4199 45.72 90)
+			(at 55.8799 29.21 90)
 			(effects
 				(font
@@
 		)
 		(property "Footprint" ""
-			(at 58.42 49.53 0)
+			(at 55.88 33.02 0)
 			(effects
 				(font
@@
 		)
 		(property "Datasheet" ""
-			(at 58.42 49.53 0)
+			(at 55.88 33.02 0)
 			(effects
 				(font
@@
 		)
 		(property "Description" "Power symbol creates a global label with name \"+5V\""
-			(at 58.42 49.53 0)
+			(at 55.88 33.02 0)
 			(effects
 				(font
@@
 	(symbol
 		(lib_id "Device:R_Small")
-		(at 58.42 54.61 0)
+		(at 55.88 38.1 0)
 		(unit 1)
 		(exclude_from_sim no)
@@
 		(dnp no)
 		(property "Reference" "R0"
-			(at 60.96 53.34 0)
+			(at 58.42 36.83 0)
 			(effects
 				(font
@@
 		)
 		(property "Value" "10k"
-			(at 60.96 55.88 0)
+			(at 58.42 39.37 0)
 			(effects
 				(font
@@
 		)
 		(property "Footprint" "Resistor_SMD:R_0805_2012Metric"
-			(at 58.42 54.61 0)
+			(at 55.88 38.1 0)
 			(effects
 				(font
@@
 		)
 		(property "Datasheet" "~"
-			(at 58.42 54.61 0)
+			(at 55.88 38.1 0)
 			(effects
 				(font
@@
 		)
 		(property "Description" "Resistor, small symbol"
-			(at 58.42 54.61 0)
+			(at 55.88 38.1 0)
 			(effects
 				(font
@@
 	(symbol
 		(lib_id "power:GND")
-		(at 46.99 63.5 0)
+		(at 40.64 43.18 0)
 		(unit 1)
 		(exclude_from_sim no)
@@
 		(fields_autoplaced yes)
 		(property "Reference" "#PWR08"
-			(at 46.99 69.85 0)
+			(at 40.64 49.53 0)
 			(effects
 				(font
@@
 		)
 		(property "Value" "GND"
-			(at 46.99 68.58 0)
+			(at 40.64 48.26 0)
 			(effects
 				(font
@@
 		)
 		(property "Footprint" ""
-			(at 46.99 63.5 0)
+			(at 40.64 43.18 0)
 			(effects
 				(font
@@
 		)
 		(property "Datasheet" ""
-			(at 46.99 63.5 0)
+			(at 40.64 43.18 0)
 			(effects
 				(font
@@
 		)
 		(property "Description" "Power symbol creates a global label with name \"GND\" , ground"
-			(at 46.99 63.5 0)
+			(at 40.64 43.18 0)
 			(effects
 				(font

Commit message: sch/pcb adjustments (UDB)
Parts:
- removed F0: 500mA, Fuse:Fuse_1206_3216Metric, symbol Device:Fuse_Small
- removed U2: SRV05-4, Package_TO_SOT_SMD:SOT-23-6, symbol marbastlib-various:SRV05-4
- J1: footprint Connector_JST:JST_EH_S4B-EH_1x04_P2.50mm_Horizontal -> Connector_JST:JST_SH_SM04B-SRSS-TB_1x04-1MP_P1.00mm_Horizontal
Connections:
- net +5V: now also J1.1 (Pin_1)
- net VBUS: no longer J1.1 (Pin_1)
- no-connect marks 6 -> 4

Commit message: BOM/CPL generated
Changed lines of the file:
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@@
 	(wire
 		(pts
-			(xy 128.27 137.16) (xy 137.16 137.16)
-		)
-		(stroke
-			(width 0)
-			(type default)
-		)
-	)
-	(wire
-		(pts
 			(xy 176.53 285.75) (xy 176.53 295.91)
 		)
@@
 	(wire
 		(pts
-			(xy 128.27 144.78) (xy 137.16 144.78)
+			(xy 128.27 137.16) (xy 137.16 137.16)
 		)
 		(stroke
@@
 	(symbol
 		(lib_id "power:GND")
-		(at 128.27 144.78 0)
+		(at 128.27 137.16 0)
 		(unit 1)
 		(exclude_from_sim no)
@@
 		(fields_autoplaced yes)
 		(property "Reference" "#PWR016"
-			(at 128.27 151.13 0)
+			(at 128.27 143.51 0)
 			(effects
 				(font
@@
 		)
 		(property "Value" "GND"
-			(at 128.27 149.86 0)
+			(at 128.27 142.24 0)
 			(effects
 				(font
@@
 		)
 		(property "Footprint" ""
-			(at 128.27 144.78 0)
+			(at 128.27 137.16 0)
 			(effects
 				(font
@@
 		)
 		(property "Datasheet" ""
-			(at 128.27 144.78 0)
+			(at 128.27 137.16 0)
 			(effects
 				(font
@@
 		)
 		(property "Description" "Power symbol creates a global label with name \"GND\" , ground"
-			(at 128.27 144.78 0)
+			(at 128.27 137.16 0)
 			(effects
 				(font
@@
 	(symbol
 		(lib_id "power:PWR_FLAG")
-		(at 137.16 144.78 0)
+		(at 137.16 137.16 0)
 		(unit 1)
 		(exclude_from_sim no)
@@
 		(fields_autoplaced yes)
 		(property "Reference" "#FLG02"
-			(at 137.16 142.875 0)
+			(at 137.16 135.255 0)
 			(effects
 				(font
@@
 		)
 		(property "Value" "PWR_FLAG"
-			(at 137.16 139.7 0)
+			(at 137.16 132.08 0)
 			(effects
 				(font
@@
 		)
 		(property "Footprint" ""
-			(at 137.16 144.78 0)
+			(at 137.16 137.16 0)
 			(effects
 				(font
@@
 		)
 		(property "Datasheet" "~"
-			(at 137.16 144.78 0)
+			(at 137.16 137.16 0)
 			(effects
 				(font
@@
 		)
 		(property "Description" "Special symbol for telling ERC where power comes from"
-			(at 137.16 144.78 0)
+			(at 137.16 137.16 0)
 			(effects
 				(font
@@
 	)
 	(symbol
-		(lib_id "power:+5V")
-		(at 128.27 137.16 0)
-		(unit 1)
-		(exclude_from_sim no)
-		(in_bom yes)
-		(on_board yes)
-		(dnp no)
-		(fields_autoplaced yes)
-		(property "Reference" "#PWR013"
-			(at 128.27 140.97 0)
-			(effects
-				(font
-					(size 1.27 1.27)
-				)
-				(hide yes)
-			)
-		)
-		(property "Value" "VBUS"
-			(at 128.27 132.08 0)
-			(effects
-				(font
-					(size 1.27 1.27)
-				)
-			)
-		)
-		(property "Footprint" ""
-			(at 128.27 137.16 0)
-			(effects
-				(font
-					(size 1.27 1.27)
-				)
-				(hide yes)
-			)
-		)
-		(property "Datasheet" ""
-			(at 128.27 137.16 0)
-			(effects
-				(font
-					(size 1.27 1.27)
-				)
-				(hide yes)
-			)
-		)
-		(property "Description" "Power symbol creates a global label with name \"+5V\""
-			(at 128.27 137.16 0)
-			(effects
-				(font
-					(size 1.27 1.27)
-				)
-				(hide yes)
-			)
-		)
-		(pin "1"
-		)
-		(instances
-			(project "tabesco-48"
-				(path "/588218a1-c895-477e-9c13-7f6d8ca7aace"
-					(reference "#PWR013")
-					(unit 1)
-				)
-			)
-		)
-	)
-	(symbol
 		(lib_id "Device:D_Small")
 		(at 134.62 255.27 90)
@@
 					(unit 1)
 				)
-			)
-		)
-	)
-	(symbol
-		(lib_id "power:PWR_FLAG")
-		(at 137.16 137.16 0)
-		(unit 1)
-		(exclude_from_sim no)
-		(in_bom yes)
-		(on_board yes)
-		(dnp no)
-		(fields_autoplaced yes)
-		(property "Reference" "#FLG01"
-			(at 137.16 135.255 0)
-			(effects
-				(font
-					(size 1.27 1.27)
-				)
-				(hide yes)
-			)
-		)
-		(property "Value" "PWR_FLAG"
-			(at 137.16 132.08 0)
-			(effects
-				(font
-					(size 1.27 1.27)
-				)
-			)
-		)
-		(property "Footprint" ""
-			(at 137.16 137.16 0)
-			(effects
-				(font
-					(size 1.27 1.27)
-				)
-				(hide yes)
-			)
-		)
-		(property "Datasheet" "~"
-			(at 137.16 137.16 0)
-			(effects
-				(font
-					(size 1.27 1.27)
-				)
-				(hide yes)
-			)
-		)
-		(property "Description" "Special symbol for telling ERC where power comes from"
-			(at 137.16 137.16 0)
-			(effects
-				(font
-					(size 1.27 1.27)
-				)
-				(hide yes)
-			)
-		)
-		(pin "1"
-		)
-		(instances
-			(project "tabesco-48"
-				(path "/588218a1-c895-477e-9c13-7f6d8ca7aace"
-					(reference "#FLG01")
-					(unit 1)
-				)

Commit message: reorganized idk
Parts:
- MX12, MX31, MX39, MX4: footprint marbastlib-mx:SW_MX_HS_CPG151101S11_1u -> marbastlib-mx:SW_MX_HS_CPG151101S11_1.75u
- MX17, MX26, MX55, MX57: footprint marbastlib-mx:SW_MX_HS_CPG151101S11_1u -> marbastlib-mx:SW_MX_HS_CPG151101S11_1.25u
- MX44: footprint marbastlib-mx:SW_MX_HS_CPG151101S11_1u -> marbastlib-mx:SW_MX_HS_CPG151101S11_1.5u
Connections:
- net col0: now also U1.38 (PF5); no longer U1.21 (PD3)
- net col1: now also U1.39 (PF4); no longer U1.20 (PD2)
- net col10: now also U1.28 (PB4); no longer U1.30 (PB6)
- net col11: now also U1.27 (PD7); no longer U1.31 (PC6)
- net col12: now also U1.26 (PD6); no longer U1.32 (PC7)
- net col13: now also U1.25 (PD4); no longer U1.36 (PF7)
- net col2: now also U1.40 (PF1); no longer U1.19 (PD1)
- net col3: now also U1.41 (PF0); no longer U1.18 (PD0)
- net col4: now also U1.36 (PF7); no longer U1.22 (PD5)
- net col5: now also U1.37 (PF6); no longer U1.25 (PD4)
- net col6: now also U1.30 (PB6); no longer U1.26 (PD6)
- net col7: now also U1.31 (PC6); no longer U1.27 (PD7)
- net col8: now also U1.32 (PC7); no longer U1.28 (PB4)
- net row0: now also U1.18 (PD0); no longer U1.38 (PF5)
- net row1: now also U1.19 (PD1); no longer U1.37 (PF6)
- net row2: now also U1.20 (PD2); no longer U1.39 (PF4)
- net row3: now also U1.22 (PD5); no longer U1.40 (PF1)
- net row4: now also U1.21 (PD3); no longer U1.41 (PF0)
Changed lines of the file:
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@@
 	)
 	(label "col12"
-		(at 87.63 90.17 0)
+		(at 87.63 110.49 0)
 		(fields_autoplaced yes)
 		(effects
@@
 	)
 	(label "col4"
-		(at 87.63 107.95 0)
+		(at 87.63 138.43 0)
 		(fields_autoplaced yes)
 		(effects
@@
 	)
 	(label "col5"
-		(at 87.63 105.41 0)
+		(at 87.63 135.89 0)
 		(fields_autoplaced yes)
 		(effects
@@
 	)
 	(label "col1"
-		(at 87.63 100.33 0)
+		(at 87.63 130.81 0)
 		(fields_autoplaced yes)
 		(effects
@@
 	)
 	(label "row1"
-		(at 87.63 135.89 0)
+		(at 87.63 97.79 0)
 		(fields_autoplaced yes)
 		(effects
@@
 	)
 	(label "row0"
-		(at 87.63 133.35 0)
+		(at 87.63 95.25 0)
 		(fields_autoplaced yes)
 		(effects
@@
 	)
 	(label "col6"
-		(at 87.63 110.49 0)
+		(at 87.63 80.01 0)
 		(fields_autoplaced yes)
 		(effects
@@
 	)
 	(label "row3"
-		(at 87.63 128.27 0)
+		(at 87.63 107.95 0)
 		(fields_autoplaced yes)
 		(effects
@@
 	)
 	(label "col13"
-		(at 87.63 138.43 0)
+		(at 87.63 105.41 0)
 		(fields_autoplaced yes)
 		(effects
@@
 	)
 	(label "col7"
-		(at 87.63 113.03 0)
+		(at 87.63 87.63 0)
 		(fields_autoplaced yes)
 		(effects
@@
 	)
 	(label "col8"
-		(at 87.63 74.93 0)
+		(at 87.63 90.17 0)
 		(fields_autoplaced yes)
 		(effects
@@
 	)
 	(label "row2"
-		(at 87.63 130.81 0)
+		(at 87.63 100.33 0)
 		(fields_autoplaced yes)
 		(effects
@@
 	)
 	(label "col0"
-		(at 87.63 102.87 0)
+		(at 87.63 133.35 0)
 		(fields_autoplaced yes)
 		(effects
@@
 	)
 	(label "row4"
-		(at 87.63 125.73 0)
+		(at 87.63 102.87 0)
 		(fields_autoplaced yes)
 		(effects
@@
 	)
 	(label "col11"
-		(at 87.63 87.63 0)
+		(at 87.63 113.03 0)
 		(fields_autoplaced yes)
 		(effects
@@
 	)
 	(label "col10"
-		(at 87.63 80.01 0)
+		(at 87.63 74.93 0)
 		(fields_autoplaced yes)
 		(effects
@@
 	)
 	(label "col3"
-		(at 87.63 95.25 0)
+		(at 87.63 125.73 0)
 		(fields_autoplaced yes)
 		(effects
@@
 	)
 	(label "col2"
-		(at 87.63 97.79 0)
+		(at 87.63 128.27 0)
 		(fields_autoplaced yes)
 		(effects
@@
 			)
 		)
-		(property "Footprint" "marbastlib-mx:SW_MX_HS_CPG151101S11_1u"
+		(property "Footprint" "marbastlib-mx:SW_MX_HS_CPG151101S11_1.75u"
 			(at 128.27 252.73 0)
 			(effects
@@
 		(on_board yes)
 		(dnp no)
-		(fields_autoplaced yes)
 		(property "Reference" "#PWR022"
 			(at 97.79 124.46 0)
@@
 		)
 		(property "Value" "GND"
-			(at 97.79 123.19 0)
+			(at 97.79 122.428 0)
 			(effects
 				(font
@@
 			)
 		)
-		(property "Footprint" "marbastlib-mx:SW_MX_HS_CPG151101S11_1u"
+		(property "Footprint" "marbastlib-mx:SW_MX_HS_CPG151101S11_1.5u"
 			(at 128.27 283.21 0)
 			(effects
@@
 			)
 		)
-		(property "Footprint" "marbastlib-mx:SW_MX_HS_CPG151101S11_1u"
+		(property "Footprint" "marbastlib-mx:SW_MX_HS_CPG151101S11_1.25u"
 			(at 231.14 262.89 0)
 			(effects
@@
 			)
 		)
-		(property "Footprint" "marbastlib-mx:SW_MX_HS_CPG151101S11_1u"
+		(property "Footprint" "marbastlib-mx:SW_MX_HS_CPG151101S11_1.75u"
 			(at 231.14 273.05 0)
 			(effects
@@
 			)
 		)
-		(property "Footprint" "marbastlib-mx:SW_MX_HS_CPG151101S11_1u"
+		(property "Footprint" "marbastlib-mx:SW_MX_HS_CPG151101S11_1.25u"
 			(at 151.13 293.37 0)
 			(effects
@@
 			)
 		)
-		(property "Footprint" "marbastlib-mx:SW_MX_HS_CPG151101S11_1u"
+		(property "Footprint" "marbastlib-mx:SW_MX_HS_CPG151101S11_1.75u"
 			(at 231.14 252.73 0)
 			(effects
@@
 			)
 		)
-		(property "Footprint" "marbastlib-mx:SW_MX_HS_CPG151101S11_1u"
+		(property "Footprint" "marbastlib-mx:SW_MX_HS_CPG151101S11_1.25u"
 			(at 128.27 262.89 0)
 			(effects
@@
 			)
 		)
-		(property "Footprint" "marbastlib-mx:SW_MX_HS_CPG151101S11_1u"
+		(property "Footprint" "marbastlib-mx:SW_MX_HS_CPG151101S11_1.25u"
 			(at 128.27 293.37 0)
 			(effects
@@
 			)
 		)
-		(property "Footprint" "marbastlib-mx:SW_MX_HS_CPG151101S11_1u"
+		(property "Footprint" "marbastlib-mx:SW_MX_HS_CPG151101S11_1.75u"
 			(at 128.27 273.05 0)
 			(effects
